Commit message: 코드 및 스크립트 수정

File: src/yahboomcar_description/urdf/Raspbot-V2.urdf (robot description, URDF)
Before this commit: robot Raspbot-V2, 9 links, 8 joints
Joints:
- joint arm1_Joint: type continuous -> fixed
- joint arm2_Joint: type continuous -> fixed
- joint global_shutter_camera_joint: origin xyz=0.07 0 0.01 rpy=0 1.5708 0 -> xyz=0.07 0 0.035 rpy=0 1.5708 0

Commit message: chore: urdf 카메라 위치 수정
실체 카메라 위치와 비슷하게 조금 더 앞으로 이동

File: src/yahboomcar_description/urdf/Raspbot-V2.urdf (robot description, URDF)
Before this commit: robot Raspbot-V2, 9 links, 8 joints
Joints:
- joint global_shutter_camera_joint: origin xyz=0.07 0 0.035 rpy=0 1.5708 0 -> xyz=0.08 0 0.035 rpy=0 1.5708 0

Commit message: chore: 시뮬레이션 구현

File: src/yahboomcar_description/urdf/Raspbot-V2.urdf (robot description, URDF)
Before this commit: robot Raspbot-V2, 9 links, 8 joints
Joints:
- joint global_shutter_camera_joint: origin xyz=0.08 0 0.035 rpy=0 1.5708 0 -> xyz=0.08 0 0.030 rpy=0 1.5708 0

Commit message: chore: 시뮬레이션에서 nav2에 기반한 로봇 이동 확인

File: src/yahboomcar_description/urdf/Raspbot-V2.urdf (robot description, URDF)
Before this commit: robot Raspbot-V2, 9 links, 8 joints
Joints:
- joint r1_Joint: axis 0 -1 0 -> 0 1 0
- joint r2_Joint: axis 0 -1 0 -> 0 1 0
